File: led-bar.kicad_pcb (KiCad board)
At the start: 2 copper layers, 174 x 12 mm, 17 parts, among them J1 Input, J2 Output

Commit message: Further workings on final design
Routing:
- net +5V: track 188.7 -> 187.1 mm
- net Net-(D3-CO): track 22.1 -> 21.2 mm
- net /dataIn: track 5.05 -> 4.21 mm
- net Net-(D3-DO): track 21.5 -> 20.7 mm
Other:
- board text added: "led-bar (nixie-vfd-clock) v1.0 2024-04 by MG-5"
- board text removed: "led-bar (nixie-clock) v1.0 2024-03 by MG-5"
