File: high-side-switch.kicad_sch (KiCad schematic)
At the start: 6 parts, among them Q34 Q_PNP_BCE, Q7 Q_NPN_BCE

Commit message: Add PCB and update Schematic
Parts:
- removed Q34: Q_PNP_BCE, symbol Device:Q_PNP_BCE
- removed Q7: Q_NPN_BCE, symbol Device:Q_NPN_BCE
- added Q2: 2N6517BU, Package_TO_SOT_THT:TO-92_Wide, symbol Device:Q_NPN_EBC
- added Q3: 2N6520TA, Package_TO_SOT_THT:TO-92_Wide, symbol Device:Q_PNP_EBC
- R18: renamed from R12; value 10k -> 13k; footprint (none) -> Resistor_SMD:R_1206_3216Metric_Pad1.30x1.75mm_HandSolder
- R19: renamed from R13; footprint (none) -> Resistor_SMD:R_1206_3216Metric_Pad1.30x1.75mm_HandSolder
- R20: renamed from R14; value 3k9 -> 13k; footprint (none) -> Resistor_SMD:R_1206_3216Metric_Pad1.30x1.75mm_HandSolder
- R21: renamed from R15; footprint (none) -> Resistor_SMD:R_0603_1608Metric_Pad0.98x0.95mm_HandSolder
Connections:
- net Dot: now also Q3.3 (C)
- net GND: now also Q2.1 (E)
- net V_{IN}: now also Q3.1 (E)
- net at R21.2: now also Q2.2 (B)
- net at R19.1: now also Q2.3 (C)
- net at R18.1, R19.2: now also Q3.2 (B)
Other:
- note added: "due multiplexing the pulse current should be 6x 2.5mA -> 15mA"

Commit message: Update values to soldered ones
Parts:
- R20: value 13k -> 2k2
Other:
- note added: "due multiplexing the pulse current should be 6x 2.5mA -> 15mA tests shows: 2k2 -> 10mA"
- note removed: "due multiplexing the pulse current should be 6x 2.5mA -> 15mA"
Changed lines of the file:
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@@
 		)
 	)
-	(text "due multiplexing the pulse current \nshould be 6x 2.5mA -> 15mA"
+	(text "due multiplexing the pulse current \nshould be 6x 2.5mA -> 15mA\n\ntests shows: 2k2 -> 10mA"
 		(exclude_from_sim no)
 		(at 144.78 96.52 0)
@@
 			)
 		)
-		(property "Value" "13k"
+		(property "Value" "2k2"
 			(at 121.92 96.52 90)
 			(effects
