File: low-side-switch.kicad_sch (KiCad schematic)
At the start: 3 parts, among them Q15 Q_NPN_BCE

Commit message: Add PCB and update Schematic
Parts:
- removed Q15: Q_NPN_BCE, symbol Device:Q_NPN_BCE
- added Q14: 2N6517BU, Package_TO_SOT_THT:TO-92_Wide, symbol Device:Q_NPN_EBC
- R41: renamed from R35; footprint (none) -> Resistor_SMD:R_0603_1608Metric_Pad0.98x0.95mm_HandSolder
- R44: renamed from R38; footprint (none) -> Resistor_SMD:R_1206_3216Metric_Pad1.30x1.75mm_HandSolder
Connections:
- net Cathode: now also Q14.3 (C)
- net GND: now also Q14.1 (E)
- net at R41.2: now also Q14.2 (B)

Commit message: Add dimming option
Parts:
- renumbered R44 to R42
Changed lines of the file:
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@@
 					(unit 1)
 				)
-				(path "/ce257b15-bcae-43e8-9f21-6657b72a9b33/26ca3393-4042-4258-a983-a953eb687fc9"
+				(path "/ce257b15-bcae-43e8-9f21-6657b72a9b33/405c8dfa-aa44-4b06-b3e2-5c275b160ac2"
 					(reference "Q15")
 					(unit 1)
 				)
-				(path "/ce257b15-bcae-43e8-9f21-6657b72a9b33/3d2eaa1d-5ba4-4e6a-8096-33f700c25ee4"
+				(path "/ce257b15-bcae-43e8-9f21-6657b72a9b33/64bfee18-f7cb-4b24-9609-0f391cee8a67"
 					(reference "Q16")
 					(unit 1)
 				)
-				(path "/ce257b15-bcae-43e8-9f21-6657b72a9b33/31a88152-31f5-4a37-b558-d330d1f1d969"
+				(path "/ce257b15-bcae-43e8-9f21-6657b72a9b33/6d576474-1063-4288-9d12-4799785c4ed0"
 					(reference "Q17")
 					(unit 1)
 				)
-				(path "/ce257b15-bcae-43e8-9f21-6657b72a9b33/21257856-8aad-49f8-8c31-b4e86dc4eca6"
+				(path "/ce257b15-bcae-43e8-9f21-6657b72a9b33/8433f7e5-9930-4f10-b8a0-7b555bf3ff53"
 					(reference "Q18")
 					(unit 1)
 				)
-				(path "/ce257b15-bcae-43e8-9f21-6657b72a9b33/c905101c-92f7-4444-865b-ee71cb43079e"
+				(path "/ce257b15-bcae-43e8-9f21-6657b72a9b33/19f543d6-04b3-4aca-a291-78ab94ee9949"
 					(reference "Q19")
 					(unit 1)
 				)
-				(path "/ce257b15-bcae-43e8-9f21-6657b72a9b33/edf12ef7-fed8-4f76-90a4-104863964e32"
+				(path "/ce257b15-bcae-43e8-9f21-6657b72a9b33/4cb5c388-d568-4aee-b68d-360cfa0db082"
 					(reference "Q20")
 					(unit 1)
 				)
-				(path "/ce257b15-bcae-43e8-9f21-6657b72a9b33/db8e2a42-b194-43f8-9014-5cf2726bc3c5"
+				(path "/ce257b15-bcae-43e8-9f21-6657b72a9b33/04c44ae7-6464-48c2-ae43-04bc58577f3d"
 					(reference "Q21")
 					(unit 1)
 				)
-				(path "/ce257b15-bcae-43e8-9f21-6657b72a9b33/bcc3003e-5a4b-4a0d-9494-d9836d4017ba"
+				(path "/ce257b15-bcae-43e8-9f21-6657b72a9b33/06c35912-72e4-4085-954d-4c0e203c0533"
 					(reference "Q22")
 					(unit 1)
 				)
-				(path "/ce257b15-bcae-43e8-9f21-6657b72a9b33/6427122d-ca8d-458b-94e4-2742fbb00f14"
+				(path "/ce257b15-bcae-43e8-9f21-6657b72a9b33/150df97e-2711-464d-8647-731330091eab"
 					(reference "Q23")
 					(unit 1)
@@
 		(on_board yes)
 		(dnp no)
-		(property "Reference" "R44"
+		(property "Reference" "R42"
 			(at 180.34 93.98 90)
 			(effects
@@
 		(instances
 			(project "nixie-clock"
-				(path "/ce257b15-bcae-43e8-9f21-6657b72a9b33/26ca3393-4042-4258-a983-a953eb687fc9"
-					(reference "R44")
-					(unit 1)
-				)
-				(path "/ce257b15-bcae-43e8-9f21-6657b72a9b33/3d2eaa1d-5ba4-4e6a-8096-33f700c25ee4"
-					(reference "R46")
-					(unit 1)
-				)
-				(path "/ce257b15-bcae-43e8-9f21-6657b72a9b33/31a88152-31f5-4a37-b558-d330d1f1d969"
-					(reference "R48")
-					(unit 1)
-				)
-				(path "/ce257b15-bcae-43e8-9f21-6657b72a9b33/21257856-8aad-49f8-8c31-b4e86dc4eca6"
-					(reference "R50")
-					(unit 1)
-				)
-				(path "/ce257b15-bcae-43e8-9f21-6657b72a9b33/c905101c-92f7-4444-865b-ee71cb43079e"
-					(reference "R52")
-					(unit 1)
-				)
-				(path "/ce257b15-bcae-43e8-9f21-6657b72a9b33/edf12ef7-fed8-4f76-90a4-104863964e32"
-					(reference "R54")
-					(unit 1)
-				)
-				(path "/ce257b15-bcae-43e8-9f21-6657b72a9b33/db8e2a42-b194-43f8-9014-5cf2726bc3c5"
-					(reference "R56")
-					(unit 1)
-				)
-				(path "/ce257b15-bcae-43e8-9f21-6657b72a9b33/bcc3003e-5a4b-4a0d-9494-d9836d4017ba"
-					(reference "R58")
-					(unit 1)
-				)
-				(path "/ce257b15-bcae-43e8-9f21-6657b72a9b33/6427122d-ca8d-458b-94e4-2742fbb00f14"
-					(reference "R60")
-					(unit 1)
-				)
 				(path "/ce257b15-bcae-43e8-9f21-6657b72a9b33/58d4c860-da1d-472a-b89e-4f5c11c28069"
 					(reference "R42")
+					(unit 1)
+				)
+				(path "/ce257b15-bcae-43e8-9f21-6657b72a9b33/405c8dfa-aa44-4b06-b3e2-5c275b160ac2"
+					(reference "R44")
+					(unit 1)
+				)
+				(path "/ce257b15-bcae-43e8-9f21-6657b72a9b33/64bfee18-f7cb-4b24-9609-0f391cee8a67"
+					(reference "R46")
+					(unit 1)
+				)
+				(path "/ce257b15-bcae-43e8-9f21-6657b72a9b33/6d576474-1063-4288-9d12-4799785c4ed0"
+					(reference "R48")
+					(unit 1)
+				)
+				(path "/ce257b15-bcae-43e8-9f21-6657b72a9b33/8433f7e5-9930-4f10-b8a0-7b555bf3ff53"
+					(reference "R50")
+					(unit 1)
+				)
+				(path "/ce257b15-bcae-43e8-9f21-6657b72a9b33/19f543d6-04b3-4aca-a291-78ab94ee9949"
+					(reference "R52")
+					(unit 1)
+				)
+				(path "/ce257b15-bcae-43e8-9f21-6657b72a9b33/4cb5c388-d568-4aee-b68d-360cfa0db082"
+					(reference "R54")
+					(unit 1)
+				)
+				(path "/ce257b15-bcae-43e8-9f21-6657b72a9b33/04c44ae7-6464-48c2-ae43-04bc58577f3d"
+					(reference "R56")
+					(unit 1)
+				)
+				(path "/ce257b15-bcae-43e8-9f21-6657b72a9b33/06c35912-72e4-4085-954d-4c0e203c0533"
+					(reference "R58")
+					(unit 1)
+				)
+				(path "/ce257b15-bcae-43e8-9f21-6657b72a9b33/150df97e-2711-464d-8647-731330091eab"
+					(reference "R60")
 					(unit 1)
 				)
@@
 		(dnp no)
 		(fields_autoplaced yes)
-		(property "Reference" "#PWR062"
+		(property "Reference" "#PWR061"
 			(at 167.64 114.3 0)
 			(effects
@@
 		(instances
 			(project "nixie-clock"
-				(path "/ce257b15-bcae-43e8-9f21-6657b72a9b33/26ca3393-4042-4258-a983-a953eb687fc9"
-					(reference "#PWR062")
-					(unit 1)
-				)
-				(path "/ce257b15-bcae-43e8-9f21-6657b72a9b33/3d2eaa1d-5ba4-4e6a-8096-33f700c25ee4"
-					(reference "#PWR063")
-					(unit 1)
-				)
-				(path "/ce257b15-bcae-43e8-9f21-6657b72a9b33/31a88152-31f5-4a37-b558-d330d1f1d969"
-					(reference "#PWR064")
-					(unit 1)
-				)
-				(path "/ce257b15-bcae-43e8-9f21-6657b72a9b33/21257856-8aad-49f8-8c31-b4e86dc4eca6"
-					(reference "#PWR065")
-					(unit 1)
-				)
-				(path "/ce257b15-bcae-43e8-9f21-6657b72a9b33/c905101c-92f7-4444-865b-ee71cb43079e"
-					(reference "#PWR066")
-					(unit 1)
-				)
-				(path "/ce257b15-bcae-43e8-9f21-6657b72a9b33/edf12ef7-fed8-4f76-90a4-104863964e32"
-					(reference "#PWR067")
-					(unit 1)
-				)
-				(path "/ce257b15-bcae-43e8-9f21-6657b72a9b33/db8e2a42-b194-43f8-9014-5cf2726bc3c5"
-					(reference "#PWR068")
-					(unit 1)
-				)
-				(path "/ce257b15-bcae-43e8-9f21-6657b72a9b33/bcc3003e-5a4b-4a0d-9494-d9836d4017ba"
-					(reference "#PWR069")
-					(unit 1)
-				)
-				(path "/ce257b15-bcae-43e8-9f21-6657b72a9b33/6427122d-ca8d-458b-94e4-2742fbb00f14"
-					(reference "#PWR070")
-					(unit 1)
-				)
 				(path "/ce257b15-bcae-43e8-9f21-6657b72a9b33/58d4c860-da1d-472a-b89e-4f5c11c28069"
 					(reference "#PWR061")
+					(unit 1)
+				)
+				(path "/ce257b15-bcae-43e8-9f21-6657b72a9b33/405c8dfa-aa44-4b06-b3e2-5c275b160ac2"
+					(reference "#PWR062")
+					(unit 1)
+				)
+				(path "/ce257b15-bcae-43e8-9f21-6657b72a9b33/64bfee18-f7cb-4b24-9609-0f391cee8a67"
+					(reference "#PWR063")
+					(unit 1)
+				)
+				(path "/ce257b15-bcae-43e8-9f21-6657b72a9b33/6d576474-1063-4288-9d12-4799785c4ed0"
+					(reference "#PWR064")
+					(unit 1)
+				)
+				(path "/ce257b15-bcae-43e8-9f21-6657b72a9b33/8433f7e5-9930-4f10-b8a0-7b555bf3ff53"
+					(reference "#PWR065")
+					(unit 1)
+				)
+				(path "/ce257b15-bcae-43e8-9f21-6657b72a9b33/19f543d6-04b3-4aca-a291-78ab94ee9949"
+					(reference "#PWR066")
+					(unit 1)
+				)
+				(path "/ce257b15-bcae-43e8-9f21-6657b72a9b33/4cb5c388-d568-4aee-b68d-360cfa0db082"
+					(reference "#PWR067")
+					(unit 1)
+				)
+				(path "/ce257b15-bcae-43e8-9f21-6657b72a9b33/04c44ae7-6464-48c2-ae43-04bc58577f3d"
+					(reference "#PWR068")
+					(unit 1)
+				)
+				(path "/ce257b15-bcae-43e8-9f21-6657b72a9b33/06c35912-72e4-4085-954d-4c0e203c0533"
+					(reference "#PWR069")
+					(unit 1)
+				)
+				(path "/ce257b15-bcae-43e8-9f21-6657b72a9b33/150df97e-2711-464d-8647-731330091eab"
+					(reference "#PWR070")
 					(unit 1)
 				)
@@
 					(unit 1)
 				)
-				(path "/ce257b15-bcae-43e8-9f21-6657b72a9b33/26ca3393-4042-4258-a983-a953eb687fc9"
+				(path "/ce257b15-bcae-43e8-9f21-6657b72a9b33/405c8dfa-aa44-4b06-b3e2-5c275b160ac2"
 					(reference "R43")
 					(unit 1)
 				)
-				(path "/ce257b15-bcae-43e8-9f21-6657b72a9b33/3d2eaa1d-5ba4-4e6a-8096-33f700c25ee4"
+				(path "/ce257b15-bcae-43e8-9f21-6657b72a9b33/64bfee18-f7cb-4b24-9609-0f391cee8a67"
 					(reference "R45")
 					(unit 1)
 				)
-				(path "/ce257b15-bcae-43e8-9f21-6657b72a9b33/31a88152-31f5-4a37-b558-d330d1f1d969"
+				(path "/ce257b15-bcae-43e8-9f21-6657b72a9b33/6d576474-1063-4288-9d12-4799785c4ed0"
 					(reference "R47")
 					(unit 1)
 				)
-				(path "/ce257b15-bcae-43e8-9f21-6657b72a9b33/21257856-8aad-49f8-8c31-b4e86dc4eca6"
+				(path "/ce257b15-bcae-43e8-9f21-6657b72a9b33/8433f7e5-9930-4f10-b8a0-7b555bf3ff53"
 					(reference "R49")
 					(unit 1)
 				)
-				(path "/ce257b15-bcae-43e8-9f21-6657b72a9b33/c905101c-92f7-4444-865b-ee71cb43079e"
+				(path "/ce257b15-bcae-43e8-9f21-6657b72a9b33/19f543d6-04b3-4aca-a291-78ab94ee9949"
 					(reference "R51")
 					(unit 1)
 				)
-				(path "/ce257b15-bcae-43e8-9f21-6657b72a9b33/edf12ef7-fed8-4f76-90a4-104863964e32"
+				(path "/ce257b15-bcae-43e8-9f21-6657b72a9b33/4cb5c388-d568-4aee-b68d-360cfa0db082"
 					(reference "R53")
 					(unit 1)
 				)
-				(path "/ce257b15-bcae-43e8-9f21-6657b72a9b33/db8e2a42-b194-43f8-9014-5cf2726bc3c5"
+				(path "/ce257b15-bcae-43e8-9f21-6657b72a9b33/04c44ae7-6464-48c2-ae43-04bc58577f3d"
 					(reference "R55")
 					(unit 1)
 				)
-				(path "/ce257b15-bcae-43e8-9f21-6657b72a9b33/bcc3003e-5a4b-4a0d-9494-d9836d4017ba"
+				(path "/ce257b15-bcae-43e8-9f21-6657b72a9b33/06c35912-72e4-4085-954d-4c0e203c0533"
 					(reference "R57")
 					(unit 1)
 				)
-				(path "/ce257b15-bcae-43e8-9f21-6657b72a9b33/6427122d-ca8d-458b-94e4-2742fbb00f14"
+				(path "/ce257b15-bcae-43e8-9f21-6657b72a9b33/150df97e-2711-464d-8647-731330091eab"
 					(reference "R59")
 					(unit 1)

Commit message: Update values to soldered ones
Parts:
- R42: value 470k -> 220k
Changed lines of the file:
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@@
 			)
 		)
-		(property "Value" "470k"
+		(property "Value" "220k"
 			(at 180.34 96.52 90)
 			(effects
